File: KiCad/SF2000_Clockport_and_SD_LED.sch (KiCad schematic (older format))
At the start: 7 parts, among them J12 Conn_02x11_Odd_Even, U12 74HCT2G14GV,125, U14 74LVC8T245PW,118, U15 74LVC8T245PW,118

Commit message: Add 10k pull-up resistor for CP_D_OE-signal on U14
Parts:
- added R?: 10k, Resistor_SMD:R_0603_1608Metric_Pad0.98x0.95mm_HandSolder, symbol Device:R_Small
Connections:
- net 3V3: now also R?.2
- net CP_D_OE: now also R?.1
Changed lines of the file:
@@
 Text GLabel 5550 2650 0    50   Input ~ 0
 CP_D_DIR
-Text GLabel 6950 2750 2    50   Input ~ 0
+Text GLabel 7500 2750 3    50   Input ~ 0
 CP_D_OE
 Text GLabel 5450 3600 0    50   Input ~ 0
@@
 Text Notes 1900 5200 0    50   ~ 0
 Caution: These signals are +5V logic levels.
+Wire Wire Line
+	6950 2750 7700 2750
+Wire Wire Line
+	7700 2750 7700 2600
+$Comp
+L Device:R_Small R?
+U 1 1 6B25571D
+P 7700 2500
+AR Path="/6B25571D" Ref="R?"  Part="1"
+AR Path="/6AFE5B10/6B25571D" Ref="R?"  Part="1"
+AR Path="/627A6500/6B25571D" Ref="R?"  Part="1"
+F 0 "R?" H 7550 2500 50  0000 L CNN
+F 1 "10k" H 7750 2500 50  0000 L CNN
+F 2 "Resistor_SMD:R_0603_1608Metric_Pad0.98x0.95mm_HandSolder" H 7700 2500 50  0001 C CNN
+F 3 "~" H 7700 2500 50  0001 C CNN
+	1    7700 2500
+	-1   0    0    1
+$EndComp
+Text GLabel 7700 2350 1    50   Input ~ 0
+3V3
+Wire Wire Line
+	7700 2400 7700 2350
 $EndSCHEMATC

Commit message: Add JP2 and JP3 pin-header with standard 2.54 mm pin pitch
Parts:
- gave numbers to parts that had none: 1
Changed lines of the file:
@@
 AR Path="/6B25571D" Ref="R?"  Part="1"
 AR Path="/6AFE5B10/6B25571D" Ref="R?"  Part="1"
-AR Path="/627A6500/6B25571D" Ref="R?"  Part="1"
-F 0 "R?" H 7550 2500 50  0000 L CNN
+AR Path="/627A6500/6B25571D" Ref="R25"  Part="1"
+F 0 "R25" H 7500 2500 50  0000 L CNN
 F 1 "10k" H 7750 2500 50  0000 L CNN
 F 2 "Resistor_SMD:R_0603_1608Metric_Pad0.98x0.95mm_HandSolder" H 7700 2500 50  0001 C CNN

Commit message: Change C38 reference to C48, Change C40 reference to C47, Change C48 reference to C44, Change C44 reference to C43, Change C43 reference to C42, Change C42 reference to C41, Change C41 reference to C40, Change C47 reference to C39, Change C39 reference to C38.
Parts:
- renumbered C38 to C48
Changed lines of the file:
@@
 AR Path="/683D3421" Ref="C?"  Part="1"
 AR Path="/620D263D/683D3421" Ref="C?"  Part="1"
-AR Path="/627A6500/683D3421" Ref="C38"  Part="1"
-F 0 "C38" H 4250 5100 50  0000 L CNN
+AR Path="/627A6500/683D3421" Ref="C48"  Part="1"
+F 0 "C48" H 4250 5100 50  0000 L CNN
 F 1 "0.1uF" H 4200 4900 50  0000 L CNN
 F 2 "Capacitor_SMD:C_0603_1608Metric_Pad1.08x0.95mm_HandSolder" H 4238 4850 50  0001 C CNN

Commit message: Change C45 reference to C48, Change C44 reference to C47, Change C48 reference to C45, Change C47 reference to C44.
Parts:
- renumbered C48 to C45
Changed lines of the file:
@@
 AR Path="/683D3421" Ref="C?"  Part="1"
 AR Path="/620D263D/683D3421" Ref="C?"  Part="1"
-AR Path="/627A6500/683D3421" Ref="C48"  Part="1"
-F 0 "C48" H 4250 5100 50  0000 L CNN
+AR Path="/627A6500/683D3421" Ref="C45"  Part="1"
+F 0 "C45" H 4250 5100 50  0000 L CNN
 F 1 "0.1uF" H 4200 4900 50  0000 L CNN
 F 2 "Capacitor_SMD:C_0603_1608Metric_Pad1.08x0.95mm_HandSolder" H 4238 4850 50  0001 C CNN
